File: Led Board/Led Board.kicad_pcb (KiCad board)
At the start: 2 copper layers, 13 parts, among them P1 CONN_01X03, P2 CONN_01X05

Commit message: a commit from desktop
Parts:
- added C1: CP1, Capacitors_Tantalum_SMD:TantalC_SizeR_EIA-2012, F.Cu at (153.2, 76.6)
- added C2: CP1, Capacitors_Tantalum_SMD:TantalC_SizeR_EIA-2012, F.Cu at (153.2, 81.7)
- added D1: LED, LEDs:LED-3MM, F.Cu at (178.0, 56.0)
- added D2: LED, LEDs:LED-3MM, F.Cu at (178.0, 50.9)
- added D3: LED, LEDs:LED-3MM, F.Cu at (178.0, 45.8)
- added D4: LED, LEDs:LED-3MM, F.Cu at (178.0, 40.7)
- added P1: CONN_01X03, Pin_Headers:Pin_Header_Straight_1x03, F.Cu at (157.0, 81.7)
- added P2: CONN_01X05, Pin_Headers:Pin_Header_Straight_1x05, F.Cu at (165.3, 43.3)
- added R1: 330, Resistors_SMD:R_0805_HandSoldering, F.Cu at (170.4, 56.0)
- added R2: 330, Resistors_SMD:R_0805_HandSoldering, F.Cu at (170.4, 50.9)
- added R3: 330, Resistors_SMD:R_0805_HandSoldering, F.Cu at (170.4, 45.8)
- added R4: 330, Resistors_SMD:R_0805_HandSoldering, F.Cu at (170.4, 40.7)
- added VoltageReg1: AP1117, TO_SOT_Packages_SMD:SOT-223, F.Cu at (146.8, 79.2)
- moved D2 53.9 mm to (156.9, 50.5)
- moved D3 53.9 mm to (156.9, 45.4)
- moved R2 53.9 mm to (149.3, 50.5)
- moved R3 53.9 mm to (149.3, 45.4)
- moved R4 53.9 mm to (149.3, 40.3)
- moved D1 53.9 mm to (156.9, 55.6)
- moved R1 53.9 mm to (149.3, 55.6)
- moved P2 53.9 mm to (144.2, 42.9)
- moved D4 53.5 mm to (156.3, 40.3)
- moved P1 53.0 mm to (157.1, 68.3)
- moved VoltageReg1 53.0 mm to (146.9, 65.8)
- moved C1 53.0 mm to (153.3, 63.2)
- moved C2 53.0 mm to (153.3, 68.3)
Routing:
- net Net-(D1-Pad1): track 0.00 -> 56.0 mm, vias 0 -> 2
- net /Vout: track 0.00 -> 40.2 mm
- net /GND: track 0.00 -> 22.7 mm
- net /Vin: track 0.00 -> 15.9 mm
- net Net-(P2-Pad2): track 0.00 -> 13.4 mm
- net Net-(P2-Pad5): track 0.00 -> 10.9 mm
- net Net-(P2-Pad3): track 0.00 -> 9.74 mm
- net Net-(P2-Pad4): track 0.00 -> 7.46 mm
- net Net-(D4-Pad2): track 0.00 -> 7.46 mm
- net Net-(D3-Pad2): track 0.00 -> 7.46 mm
- net Net-(D2-Pad2): track 0.00 -> 7.46 mm
- net Net-(D1-Pad2): track 0.00 -> 7.46 mm
Other:
- board outline added: 100 x 100 mm
