File: Led Board/Led Board.sch (KiCad schematic (older format))
At the start: 13 parts, among them P1 CONN_01X03, P2 CONN_01X05

Commit message: a commit from desktop
Parts:
- D1, D2, D3, D4: symbol LED -> LED-RESCUE-Led_Board
Changed lines of the file:
@@
 EESchema Schematic File Version 2
+LIBS:Led Board-rescue
 LIBS:power
 LIBS:device
@@
 GND
 $Comp
-L LED D1
+L LED-RESCUE-Led_Board D1
 U 1 1 5AA4F763
 P 5600 3950
@@
 $EndComp
 $Comp
-L LED D2
+L LED-RESCUE-Led_Board D2
 U 1 1 5AA4F9D4
 P 6050 3950
@@
 $EndComp
 $Comp
-L LED D3
+L LED-RESCUE-Led_Board D3
 U 1 1 5AA4FB30
 P 6450 3950
@@
 $EndComp
 $Comp
-L LED D4
+L LED-RESCUE-Led_Board D4
 U 1 1 5AA4FB3C
 P 6900 3950
